Commit message: B2: real-weight mass correction, rear-stand v4/v5, jump anti-blowup fixes, new leg-lift task
- b2_description.urdf: rescaled all link masses/inertias to the real
  measured B2 weight (73.55kg with battery, was 74.58kg) so training and
  the MuJoCo bench agree on mass.
- rear_stand: v4 adds a gait-phase clock (sin/cos command slots) and real
  turning (yaw command slot), ported from workshop_legged_gym's go2_stand.
  v5 redesigns the walking economics after a bench test showed the v4
  final checkpoint stands but never walks: more walk-command exposure per
  cycle, a slower gait-clock frequency matched to B2's mass, command
  magnitudes that don't let standing-still masquerade as tracking, and
  rebalanced gait-mechanism reward weights. action_rate_l2 gets a
  rear_stand-only clamped override after two live vloss-blowup incidents
  traced to an unbounded squared penalty.
- jump: clamped motor_speed_violation/airborne_leg_stillness penalties
  (same unbounded-squared-term postmortem as rear_stand's action_rate_l2),
  an idle left-right symmetry term, and a flight/landing symmetry term
  added after a bench test showed a chronic asymmetric tuck surviving
  into flight and touchdown.
- leg_lift: new task (single-leg lift command, tripod support reward) plus
  two fixes from its own first bench test — a foot-horizontal penalty so
  lifting can't be satisfied by sweeping the leg back, and a base-height
  anchor so lifting can't be satisfied by squatting.

File: source/robot_lab/data/Robots/unitree/b2_description/urdf/b2_description.urdf (robot description, URDF)
Before this commit: robot b2_description, 37 links, 36 joints
Links:
- link FL_calf: mass 0.404 -> 0.3984188854
- link FL_calf_rotor: mass 0.2734 -> 0.2696230774
- link FL_foot: mass 0.126 -> 0.1242593554
- link FL_hip: mass 2.673 -> 2.636073467
- link FL_hip_rotor: mass 0.2734 -> 0.2696230774
- link FL_thigh: mass 4.536 -> 4.473336793
- link FL_thigh_rotor: mass 0.2734 -> 0.2696230774
- link FR_calf: mass 0.404 -> 0.3984188854
- link FR_calf_rotor: mass 0.2734 -> 0.2696230774
- link FR_foot: mass 0.126 -> 0.1242593554
- link FR_hip: mass 2.673 -> 2.636073467
- link FR_hip_rotor: mass 0.2734 -> 0.2696230774
- link FR_thigh: mass 4.536 -> 4.473336793
- link FR_thigh_rotor: mass 0.2734 -> 0.2696230774
- link RL_calf: mass 0.404 -> 0.3984188854
- link RL_calf_rotor: mass 0.2734 -> 0.2696230774
- link RL_foot: mass 0.126 -> 0.1242593554
- link RL_hip: mass 2.673 -> 2.636073467
- link RL_hip_rotor: mass 0.2734 -> 0.2696230774
- link RL_thigh: mass 4.536 -> 4.473336793
- link RL_thigh_rotor: mass 0.2734 -> 0.2696230774
- link RR_calf: mass 0.404 -> 0.3984188854
- link RR_calf_rotor: mass 0.2734 -> 0.2696230774
- link RR_foot: mass 0.126 -> 0.1242593554
- link RR_hip: mass 2.673 -> 2.636073467
- link RR_hip_rotor: mass 0.2734 -> 0.2696230774
- link RR_thigh: mass 4.536 -> 4.473336793
- link RR_thigh_rotor: mass 0.2734 -> 0.2696230774
- link base_link: mass 35.86 -> 35.36460701
- link f_dc_link: mass 4.19E-15 -> 4.132116658e-15
- link f_oc_link: mass 4.19E-15 -> 4.132116658e-15
- link head_Link: mass 3.6885 -> 3.6375447
- link imu_link: mass 4.19E-15 -> 4.132116658e-15
- link lidar_link: mass 4.19E-15 -> 4.132116658e-15
- link r_dc_link: mass 4.19E-15 -> 4.132116658e-15
- link r_oc_link: mass 4.19E-12 -> 4.132116658e-12
- link tail_link: mass 0.795 -> 0.7840173612
